File: V2.x/Light/LOCO-Light.sch (EAGLE design)
At the start: 54 parts, among them IC1 Atmega 328-P, IC2 MCP2515, IC3 ACS712ELCTR-20A-T, IC5 LM340MP-05, J1 3-794618-4, J2 3-794618-4, Q1 8MHz, Q2 16MHz, Q3 FDS5680, Q4 FDS5680, Q5 FDS5680, Q6 FDS5680, Q7 FDS5680, Q8 FDS5680

Commit message: Signed-off-by: Thomas Winkler <thomas.winkler@iggmp.net>
Parts:
- removed D1, D2, D3, D4, D5, D6: BAS40, diode:BAS40
- removed LIGHT: 22-23-2071, con-molex:22-23-2071
- added CAN: GRN, led:LEDCHIP-LED0603
- added R16: 10k, rcl:R-EU_R0603
- added SDI: (no value), jumper:SJ
- added SI, SK, SO: PTR1B1,27, testpad:PTR1B1,27
- added X1: 22-23-2081, con-molex:22-23-2081
- +5V: value (none) -> GRN
Connections:
- removed net A1: IC1.PC1(ADC1)
- removed net A2: IC1.PC2(ADC2)
- removed net A3: IC1.PC3(ADC3)
- removed net A4: IC1.PC4(ADC4/SDA)
- removed net A5: IC1.PC5(ADC5/SCL)
- removed net D8: IC1.PB0(ICP)
- new net CAN-CS: IC2.!CS, SDI.2
- new net N$9: CAN.C, R16.1
- net +12V: now also X1-1.S
- net CS: now also SDI.1; no longer IC2.!CS
- net D9: now also CAN.A
- net GND: now also R16.2, X1-8.S; no longer LIGHT-7.S
- net L1: now also X1-2.S; no longer D1.C, LIGHT-1.S
- net L2: now also X1-3.S; no longer D2.C, LIGHT-2.S
- net L3: now also X1-4.S; no longer D3.C, LIGHT-3.S
- net L4: now also X1-5.S; no longer D4.C, LIGHT-4.S
- net L5: now also X1-6.S; no longer D5.C, LIGHT-5.S
- net L6: now also X1-7.S; no longer D6.C, LIGHT-6.S
- net LIGHT-GND: no longer D1.A, D2.A, D3.A, D4.A, D5.A, D6.A
- net RX: now also SV1.2; no longer SV1.3
- net SCK: now also SK.TP
- net SI: now also SI.TP
- net SO: now also SO.TP
- net TX: now also SV1.3; no longer SV1.2
Other:
- note added: "LOCO-Light V2.1a"
- moved on the sheet: Q3, Q4, Q5, Q6, Q7, Q8, R10, R11, R12, R13, R14, R3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
