File: V2.x/Light/LOCO-Light.brd (EAGLE design)
At the start: 43.2 x 34.3 mm, 54 parts, among them IC1 Atmega 328-P, IC2 MCP2515, IC3 ACS712ELCTR-20A-T, IC5 LM340MP-05, J1 3-794618-4, J2 3-794618-4, Q1 8MHz, Q2 16MHz, Q3 FDS5680, Q4 FDS5680, Q5 FDS5680, Q6 FDS5680, Q7 FDS5680, Q8 FDS5680

Commit message: Signed-off-by: Thomas Winkler <thomas.winkler@iggmp.net>
Parts:
- removed D1, D2, D3, D4, D5, D6: BAS40, diode:SOT23
- removed LIGHT: 22-23-2071, con-molex:22-23-2071
- added CAN: GRN, led:CHIP-LED0603
- added R16: 10k, rcl:R0603
- added SDI: (no value), jumper:SJ
- added SI, SK, SO: PTR1B1,27, testpad:B1,27
- added X1: 22-23-2081, con-molex:22-23-2081
- +5V: value (none) -> GRN
- moved IC3 8.90 mm to (24.1, 28.9)
- moved C14 6.98 mm to (14.0, 30.8)
- moved C15 6.98 mm to (14.0, 27.3)
- moved C16 6.04 mm to (17.8, 29.2)
- moved R1 5.40 mm to (17.5, 24.1), turned to 0 degrees
- moved R2 4.93 mm to (25.7, 22.9), turned to 90 degrees
- moved R11 3.24 mm to (30.5, 31.4)
- moved R3 3.24 mm to (34.3, 11.1)
- moved R5 3.24 mm to (34.3, 31.4)
- moved R9 3.24 mm to (30.5, 11.1)
- moved R10 3.24 mm to (30.5, 21.3)
- moved R4 3.24 mm to (34.3, 21.3)
- moved Q3 3.24 mm to (32.4, 6.03)
- moved Q4 3.24 mm to (32.4, 16.2)
- moved Q5 3.24 mm to (32.4, 26.4)
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Connections:
- removed net A1: IC1.24
- removed net A2: IC1.25
- removed net A3: IC1.26
- removed net A4: IC1.27
- removed net A5: IC1.28
- removed net D8: IC1.12
- new net CAN-CS: IC2.18, SDI.2
- new net N$9: CAN.C, R16.1
- net +12V: now also X1.1
- net CS: now also SDI.1; no longer IC2.18
- net D9: now also CAN.A
- net GND: now also R16.2, X1.8; no longer LIGHT.7
- net L1: now also X1.2; no longer D1.3, LIGHT.1
- net L2: now also X1.3; no longer D2.3, LIGHT.2
- net L3: now also X1.4; no longer D3.3, LIGHT.3
- net L4: now also X1.5; no longer D4.3, LIGHT.4
- net L5: now also X1.6; no longer D5.3, LIGHT.5
- net L6: now also X1.7; no longer D6.3, LIGHT.6
- net LIGHT-GND: no longer D1.1, D2.1, D3.1, D4.1, D5.1, D6.1
- net RX: now also SV1.2; no longer SV1.3
- net SCK: now also SK.TP
- net SI: now also SI.TP
- net SO: now also SO.TP
- net TX: now also SV1.3; no longer SV1.2
Routing:
- net D6: track 14.2 -> 82.5 mm, vias 0 -> 2
- net LIGHT-GND: track 134.5 -> 71.4 mm, vias 1 -> 3
- net +12V: track 40.8 -> 77.8 mm, vias 2 -> 1
- net D3: track 51.0 -> 19.9 mm
- net D9: track 0.00 -> 25.0 mm, vias 0 -> 3
- net VCC: track 140.0 -> 116.3 mm, vias 7 -> 8
- net GND: track 220.1 -> 242.4 mm, vias 9 -> 4
- net CAN-L: track 25.4 -> 34.8 mm, vias 2 -> 0
- net SI: track 4.19 -> 11.9 mm
- net N$9: track 0.00 -> 7.42 mm
- net SO: track 4.04 -> 10.8 mm
- net L3: track 20.9 -> 14.6 mm
- net N$15: track 30.3 -> 24.0 mm, vias 1 -> 3
- net SCK: track 2.87 -> 8.81 mm, vias 1 -> 2
- net L2: track 14.8 -> 9.56 mm
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Other:
- board text added: "+12V"
- board text added: "L3"
- board text added: "V2.1a-s"
- board text removed: "L1"
- board text removed: "L5"
- board text removed: "V 2.0"
- board text removed: "V2.1"
