File: V2.x/Motorsteuerung/Leistungsstufe.brd (EAGLE design)
At the start: 63.5 x 64.8 mm, 40 parts, among them Q1 IRF740, Q2 IRF740, Q3 IRF740, Q4 IRF740, X1 MKDSN1,5/4-5,08

Commit message: initial
Parts:
- D3, D4, D5: value (none) -> 1N4148
Connections:
- net VOLT-1: now also BUS2B.1; no longer BUS1.7
- net VOLT-2: now also BUS2B.2; no longer BUS1.8
Routing:
- net VOLT-2: track 14.4 -> 69.8 mm
- net FORWARD: track 23.9 -> 46.2 mm, vias 1 -> 0
- net VOLT-1: track 22.3 -> 38.9 mm
- net GND: track 309.2 -> 296.1 mm, vias 1 -> 0
- net MOTOR+: track 64.8 -> 67.6 mm
- net EN-MOTOR: track 17.7 -> 15.4 mm, vias 1 -> 0
- net REWARD: track 23.6 -> 21.7 mm, vias 0 -> 1
- net DRIVE: track 85.2 -> 84.6 mm
- net BREAK: track 84.1 -> 84.4 mm, vias 4 -> 5
Other:
- board text added: "LOCO-Driver"
- board text added: "V2.0a"
