File: V2.x/Motorsteuerung/Leistungsstufe.sch (EAGLE design)
At the start: 40 parts, among them Q1 IRF740, Q2 IRF740, Q3 IRF740, Q4 IRF740, X1 MKDSN1,5/4-5,08

Commit message: initial
Parts:
- D3, D4, D5: value (none) -> 1N4148
Connections:
- net VOLT-1: now also BUS2B.1; no longer BUS1.7
- net VOLT-2: now also BUS2B.2; no longer BUS1.8
Other:
- note added: "CAN-Motor-Driver V2.0a"
Changed lines of the file:
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@@
 <part name="D1" library="diode" library_urn="urn:adsk.eagle:library:210" deviceset="PBYR635" device="" package3d_urn="urn:adsk.eagle:package:43387/1"/>
 <part name="D2" library="diode" library_urn="urn:adsk.eagle:library:210" deviceset="PBYR635" device="" package3d_urn="urn:adsk.eagle:package:43387/1"/>
-<part name="D3" library="diode" library_urn="urn:adsk.eagle:library:210" deviceset="DIODE-" device="SOD323-R" package3d_urn="urn:adsk.eagle:package:43437/1"/>
-<part name="D4" library="diode" library_urn="urn:adsk.eagle:library:210" deviceset="DIODE-" device="SOD323-R" package3d_urn="urn:adsk.eagle:package:43437/1"/>
-<part name="D5" library="diode" library_urn="urn:adsk.eagle:library:210" deviceset="DIODE-" device="SOD323-R" package3d_urn="urn:adsk.eagle:package:43437/1"/>
+<part name="D3" library="diode" library_urn="urn:adsk.eagle:library:210" deviceset="DIODE-" device="SOD323-R" package3d_urn="urn:adsk.eagle:package:43437/1" value="1N4148"/>
+<part name="D4" library="diode" library_urn="urn:adsk.eagle:library:210" deviceset="DIODE-" device="SOD323-R" package3d_urn="urn:adsk.eagle:package:43437/1" value="1N4148"/>
+<part name="D5" library="diode" library_urn="urn:adsk.eagle:library:210" deviceset="DIODE-" device="SOD323-R" package3d_urn="urn:adsk.eagle:package:43437/1" value="1N4148"/>
 <part name="GND8" library="supply1" library_urn="urn:adsk.eagle:library:371" deviceset="GND" device=""/>
 <part name="R14" library="rcl" library_urn="urn:adsk.eagle:library:334" deviceset="R-EU_" device="MELF0102W" package3d_urn="urn:adsk.eagle:package:23588/2" value="47K"/>
@@
 <text x="76.2" y="17.78" size="1.778" layer="97">Freilaufdioden</text>
 <text x="104.14" y="17.78" size="1.778" layer="97">Spannungsmessung</text>
+<text x="-96.52" y="93.98" size="5.08" layer="95">CAN-Motor-Driver V2.0a</text>
 </plain>
 <instances>
@@
 <net name="VOLT-1" class="0">
 <segment>
-<pinref part="BUS1" gate="1" pin="7"/>
-<wire x1="-88.9" y1="60.96" x2="-73.66" y2="60.96" width="0.1524" layer="91"/>
-<label x="-73.66" y="60.96" size="1.778" layer="95" rot="R180"/>
-</segment>
-<segment>
 <pinref part="D6" gate="G$1" pin="C"/>
 <pinref part="R14" gate="G$1" pin="1"/>
@@
 <label x="104.14" y="10.16" size="1.778" layer="95"/>
 </segment>
+<segment>
+<pinref part="BUS2B" gate="1" pin="1"/>
+<wire x1="-88.9" y1="22.86" x2="-73.66" y2="22.86" width="0.1524" layer="91"/>
+<label x="-73.66" y="22.86" size="1.778" layer="95" rot="R180"/>
+</segment>
 </net>
 <net name="VOLT-2" class="0">
-<segment>
-<pinref part="BUS1" gate="1" pin="8"/>
-<wire x1="-88.9" y1="58.42" x2="-73.66" y2="58.42" width="0.1524" layer="91"/>
-<label x="-73.66" y="58.42" size="1.778" layer="95" rot="R180"/>
-</segment>
 <segment>
 <pinref part="D7" gate="G$1" pin="C"/>
@@
 <label x="104.14" y="-15.24" size="1.778" layer="95"/>
 </segment>
+<segment>
+<pinref part="BUS2B" gate="1" pin="2"/>
+<wire x1="-88.9" y1="20.32" x2="-73.66" y2="20.32" width="0.1524" layer="91"/>
+<label x="-73.66" y="20.32" size="1.778" layer="95" rot="R180"/>
+</segment>
 </net>
 </nets>
 </sheet>
 </sheets>
+<errors>
+</errors>
 </schematic>
 </drawing>
