File: V2.x/Sensor/LOCO-Sensor.brd (EAGLE design)
At the start: 66 x 34.3 mm, 48 parts, among them IC1 Atmega 328-P, IC2 MCP2515, IC3 LM340MP-05, IC5 ACS750LCA-050, Q1 8MHz, Q2 16MHz

Commit message: Signed-off-by: Thomas Winkler <thomas.winkler@iggmp.net>
Parts:
- removed C+-BOT, C+TOP, C-BOT, C-TOP: PAD 5.5, holes:5,5-PAD
- removed C17: 1n, rcl:C0402K
- removed C7: 100n, rcl:C0402K
- removed D1, D2, D3, D4: (no value), diode:SOD80C
- removed IC3: LM340MP-05, linear:SOT223
- removed IC5: ACS750LCA-050, allegro:ACS75050
- removed R10, R11, R4, R6, R8: 10k, rcl:MINI_MELF-0102W
- removed R3, R5, R7, R9: 220K, rcl:MINI_MELF-0102W
- removed SPEED: 1445055-2, con-amp:1445055-2
- removed VOLT: 22-23-2041, con-molex:22-23-2041
- added BUS: (no value), con-lstb:MA09-2
- added IC4: LD117AS12TR, v-reg:SOT223
- added PWR: 22-23-2021, con-molex:22-23-2021
- moved C8 8.35 mm to (25.4, 14.6)
- moved Q1 8.35 mm to (25.4, 14.6)
- moved C1 8.35 mm to (25.4, 19.4)
- moved C2 8.35 mm to (25.4, 9.84)
Connections:
- removed net C+: C-BOT.B5,5, C-TOP.B5,5, IC5.IP-, IC5.IP-@10, IC5.IP-@11, IC5.IP-@12, IC5.IP-@13, IC5.IP-@14, IC5.IP-@15, IC5.IP-@16, IC5.IP-@17, IC5.IP-@2, IC5.IP-@3, IC5.IP-@4, IC5.IP-@5, IC5.IP-@6, IC5.IP-@7, IC5.IP-@8, IC5.IP-@9
- removed net C-: C+-BOT.B5,5, C+TOP.B5,5, IC5.IP+, IC5.IP+@10, IC5.IP+@11, IC5.IP+@12, IC5.IP+@13, IC5.IP+@14, IC5.IP+@15, IC5.IP+@16, IC5.IP+@17, IC5.IP+@2, IC5.IP+@3, IC5.IP+@4, IC5.IP+@5, IC5.IP+@6, IC5.IP+@7, IC5.IP+@8, IC5.IP+@9
- removed net V1: R3.2, VOLT.1
- removed net V2: R5.2, VOLT.2
- removed net V3: R7.2, VOLT.3
- removed net V4: R9.2, VOLT.4
- new net 12V-PWR: BUS.17, PWR.1
- net +12V: now also IC4.3; no longer IC3.1
- net A0: now also BUS.13; no longer C17.2, IC5.3
- net A1: now also BUS.11; no longer D1.C, R3.1, R4.2
- net A2: now also BUS.9; no longer D2.C, R5.1, R6.2
- net A3: now also BUS.7; no longer D3.C, R7.1, R8.2
- net A4: now also BUS.5; no longer D4.C, R10.2, R9.1
- net A5: now also BUS.3
- net D2: now also BUS.2; no longer R11.2, SPEED.1
- net D3: now also BUS.4
- net D4: now also BUS.6
- net D5: now also BUS.8
- net D6: now also BUS.10
- net D7: now also BUS.12
- net D8: now also BUS.14
- net D9: now also BUS.15
- net GND: now also BUS.16, BUS.18, IC4.1, PWR.2; no longer C17.1, C7.1, D1.A, D2.A, D3.A, D4.A, IC3.4, IC5.2, R10.1, R4.1, R6.1, R8.1, SPEED.2
- net VCC: now also BUS.1, IC4.4; no longer C7.2, IC3.3, IC5.1, R11.1
Routing:
- net GND: track 251.7 -> 145.7 mm, vias 1 -> 3
- net A3: track 47.6 -> 15.7 mm, vias 0 -> 1
- net A5: track 0.00 -> 31.4 mm, vias 0 -> 2
- net D3: track 0.00 -> 29.9 mm, vias 0 -> 1
- net 12V-PWR: track 0.00 -> 29.1 mm, vias 0 -> 2
- net D4: track 0.00 -> 27.7 mm, vias 0 -> 2
- net D2: track 47.2 -> 20.4 mm, vias 1 -> 2
- net D8: track 0.00 -> 25.2 mm, vias 0 -> 1
- net D5: track 0.00 -> 24.4 mm, vias 0 -> 2
- net VCC: track 120.2 -> 143.7 mm, vias 4 -> 9
- net A2: track 26.0 -> 47.3 mm, vias 4 -> 7
- net D6: track 0.00 -> 20.5 mm, vias 0 -> 1
- net V2: track 18.6 -> 0.00 mm
- net V4: track 18.1 -> 0.00 mm
- net D7: track 0.00 -> 17.3 mm, vias 0 -> 1
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- removed copper zone on layer 1, net C+
- removed copper zone on layer 16, net C+
- removed copper zone on layer 1, net C-
- removed copper zone on layer 16, net C-
Other:
- board size 66 x 34.3 mm -> 34.3 x 34.3 mm
- board text added: "LOCO-Universal"
- board text added: "V2.0"
- board text removed: "LOCO-Sensor"
- board text removed: "V2.1"
