File: V2.x/Motor/Motor.brd (EAGLE design)
At the start: 43.2 x 34.3 mm, 41 parts, among them IC1 Atmega 328-P, IC2 MCP2515, IC3 LM340MP-05, Q1 8MHz, Q2 16MHz

Commit message: initial
Parts:
- added D4, D5: 5,1V, diode:SOD80C
- added P1: (no value), jst-ph:JST-PH2
- added R10, R8: 47K, rcl:MINI_MELF-0102W
- added R11, R9: 10k, rcl:MINI_MELF-0102W
- moved C8 1.91 mm to (16.2, 6.67)
Connections:
- new net A2: D4.C, IC1.25, R8.1, R9.2
- new net A3: D5.C, IC1.26, R10.1, R11.2
- new net BATT-1: P1.1, R8.2
- new net BATT-2: P1.2, R10.2
- net GND: now also D4.A, D5.A, R11.1, R9.1
Routing:
- net SCK: track 11.0 -> 51.6 mm, vias 2 -> 1
- net A3: track 0.00 -> 35.6 mm
- net GND: track 199.6 -> 226.9 mm, vias 1 -> 0
- net D3: track 38.8 -> 24.9 mm, vias 1 -> 2
- net A2: track 0.00 -> 13.6 mm
- net D2: track 32.0 -> 44.7 mm, vias 0 -> 1
- net A0: track 17.7 -> 29.7 mm
- net D7: track 22.7 -> 33.0 mm, vias 2 -> 3
- net RST: track 41.0 -> 49.1 mm, vias 4 -> 3
- net VCC: track 109.9 -> 115.7 mm
- net CAN-OCC1: track 19.4 -> 24.7 mm
- net N$6: track 11.6 -> 15.6 mm
- net BATT-2: track 0.00 -> 3.84 mm
- net BATT-1: track 0.00 -> 3.64 mm
- net TX: track 11.0 -> 13.0 mm, vias 1 -> 0
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- removed copper zone on layer 1, net GND
- removed copper zone on layer 16, net GND
Other:
- board text added: "V2.2-s"
- board text removed: "V2.1b-s"

Commit message: initial
Routing:
- added copper zone on layer 1, net GND
- added copper zone on layer 16, net GND
