File: V2.x/Motor/Motor.sch (EAGLE design)
At the start: 41 parts, among them IC1 CP2102, IC2 LD117AS33TR, IC3 LD117ADT50TR, IC4 MAX3468CSA, U1 ESP-WROOM-32

Commit message: Signed-off-by: Thomas Winkler <thomas.winkler@iggmp.net>
Parts:
- removed 3,3V, 5V, RX, TX: (no value), led:LED
- removed 6-30V: 22-23-2021, con-molex:22-23-2021
- removed C10, C7: 100nF, rcl:C-EUC0402
- removed IC4: MAX3468CSA, maxim:MAX3468CSA
- removed R10, R9: 20K, rcl:R-EU_MELF0102R
- removed R11: 120R, rcl:R-EU_MELF0102R
- removed R12, R8: 10K, rcl:R-EU_MELF0102R
- removed RS-485: (no value), con-subd:F09H
- removed S1: (no value), switch:255SB
- removed SV1: (no value), con-lstb:MA08-2
- removed U1: ESP-WROOM-32, esp32:ESP-WROOM-32
- removed UBS-B: (no value), con-berg:PN61729
- added +5V, CAN: (no value), led:LEDCHIP-LED0603
- added C14: 1n, rcl:C-EUC0402K
- added C15, C8: 100n, rcl:C-EUC0402K
- added C16: 16uF, rcl:CPOL-EUA/3216-18W
- added D2: 5,1V, diode:ZENER-DIODESOD80C
- added D3: 5A, diode:DIODE-DO214AA
- added DRIVER: 4-794620-0, 4-794620-0:4-794620-0
- added PROG: (no value), con-lstb:MA05-1
- added Q1: 8MHz, crystal:CRYSTALHC49S
- added Q2: 16MHz, crystal:CRYSTALHC49S
- added R15: 220R, rcl:R-EU_R0805
- added RST, SC, SI, SO: PTR1B1,27, testpad:PTR1B1,27
- added SS: 0R-JUMPA, jump-0r-smd:0R-JUMPA
- C1: value 47uF -> 22p; device rcl:CPOL-EUB/3528-21R -> rcl:C-EUC0402K
- C11: value 47uF -> 100n; device rcl:CPOL-EUB/3528-21R -> rcl:C-EUC0402K
- C12: value 100nF -> 1n; device rcl:C-EUC0402 -> rcl:C-EUC0402K
- C13: value 47uF -> 16uF; device rcl:CPOL-EUB/3528-21R -> rcl:CPOL-EUA/3216-18W
- C2, C4: value 104 -> 22p; device rcl:C-EUC0402 -> rcl:C-EUC0402K
- C3: value 47uF -> 22p; device rcl:C-EUC0402 -> rcl:C-EUC0402K
- C5: value 1uF -> 100n; device rcl:C-EUC0402 -> rcl:C-EUC0402K
- C6: device rcl:C-EUC0402 -> rcl:C-EUC0402K
- D1: value (none) -> 5,1V; device diode:DIODE-DO-214AC -> diode:ZENER-DIODESOD80C
- DA1: value TJA1050 -> MCP2551
- IC1: value CP2102 -> Atmega 328-P; device silabs:CP2102 -> atmel:MEGA8-AI
- IC2: value LD117AS33TR -> MCP2515; device v-reg:LD117AS33TR -> mcp2514:MCP2515
- IC3: value LD117ADT50TR -> LM340MP-05; device v-reg:LD117ADT50TR -> linear:LM340MP-05
- R1: value 5k -> 10k; device rcl:R-EU_MELF0102R -> rcl:R-EU_R0805
- R2: value 330R -> 10k; device rcl:R-EU_MELF0102R -> rcl:R-EU_R0805
- R3: value 330R -> 47K; device rcl:R-EU_MELF0102R -> rcl:R-EU_MELF0102W
- R4, R6: value 10K -> 10k; device rcl:R-EU_MELF0102R -> rcl:R-EU_MELF0102W
- R5: value 10K -> 47K; device rcl:R-EU_MELF0102R -> rcl:R-EU_MELF0102W
- R7: value 10K -> 220R; device rcl:R-EU_MELF0102R -> rcl:R-EU_R0805
Connections:
- net N$8 renamed CAN-H
- net N$9 renamed CAN-L
- removed net +3V3: C10.1, C11.+, C2.1, C6.1, IC1.VDD, IC2.OUT, R1.2, R4.2, R5.2, R6.2, R7.2, R8.2, SV1.1, U1.3V3
- removed net +5V: C12.1, C13.+, C3.1, CAN-1.4, CAN-2.4, DA1.VSS, IC1.REGIN, IC1.VBUS, IC3.OUT, IC4.VCC, R12.2, R9.2, RS-485.6, UBS-B.1
- removed net CAN-RX: DA1.RXD
- removed net CAN-TX: DA1.TXD
- removed net CP-CTS: IC1.CTS, U1.IO15
- removed net CP-RDX: IC1.RXD, RX.A, U1.RXD0
- removed net CP-RTS: IC1.RTS, U1.IO13
- removed net CP-TDX: IC1.TXD, TX.A, U1.TXD0
- removed net IO0: SV1.4, U1.IO0
- removed net IO14: SV1.15, U1.IO14
- removed net IO16: SV1.8, U1.IO16
- removed net IO17: SV1.10, U1.IO17
- removed net IO18: SV1.14
- removed net IO19: U1.IO19
- removed net IO2: SV1.2, U1.IO2
- removed net IO25: SV1.9, U1.IO25
- removed net IO26: SV1.11, U1.IO26
- removed net IO27: SV1.13, U1.IO27
- removed net IO32: SV1.7, U1.IO32
- removed net IO33: U1.IO33
- removed net IO34: SV1.3, U1.IO34
- removed net IO35: SV1.5, U1.IO35
- removed net IO4: SV1.6, U1.IO4
- removed net IO5: SV1.12, U1.IO5
- removed net MISO: U1.IO23
- removed net MOSI: U1.IO22
- removed net N$13: 5V.A, R12.1
- removed net N$30: U1.IO21
- removed net N$4: 6-30V-1.S, D1.A
- removed net N$5: R2.1, TX.C
- removed net N$7: R3.1, RX.C
- removed net RDX1: IC4.DI, R8.1, U1.SD2
- removed net RE/DE: IC4.DE, IC4.RE/, R6.1, R7.1, U1.IO12
- removed net RESET: C5.1, U1.EN
- removed net TDX1: IC4.RO, R5.1, U1.SD3
- new net A0: D1.C, IC1.PC0(ADC0), R3.1, R4.2
- new net A1: D2.C, IC1.PC1(ADC1), R5.1, R6.2
- new net CAN-CS: IC2.!CS, SS-0R.2
- new net CAN-OCC1: C1.1, IC2.OSC1, Q1.1
- new net CAN-OCC2: C2.1, IC2.OSC2, Q1.2
- new net CS: IC1.PB2(SS/OC1B), SS-0R.3
- new net D2: DRIVER.2, IC1.PD2(INT0)
- new net D3: DRIVER.4, IC1.PD3(INT1)
- new net D6: DRIVER.5, IC1.PD6(AIN0)
- new net D7: DRIVER.7, IC1.PD7(AIN1)
- new net D8: DRIVER.9, IC1.PB0(ICP)
- new net D9: DRIVER.3, IC1.PB1(OC1A)
- new net DTR: C8.1, PROG.1
- new net MI: IC1.PB4(MISO), IC2.SO, SI.TP
- new net MO: IC1.PB3(MOSI/OC2), IC2.SI, SO.TP
- new net MOTOR+: DRIVER.6, R3.2
- new net MOTOR-: DRIVER.8, R5.2
- new net RST: C8.2, IC1.PC6(/RESET), R2.1, RST.TP
- new net RX: IC1.PD1(TXD), PROG.2
- new net RXCAN: DA1.RXD, IC2.RXCAN
- new net TX: IC1.PD0(RXD), PROG.3
- new net TXCAN: DA1.TXD, IC2.TXCAN
- new net VCC: +5V.A, C14.2, C15.2, C16.+, C5.2, C6.1, DA1.VDD, IC1.AVCC, IC1.VCC@1, IC2.VDD, IC3.VO, PROG.4, R1.2, R2.2, SS-0R.1
- net +12V: now also C11.2, C12.2, C13.+, CAN-1.4, CAN-2.4, D3.C, IC3.VI; no longer C1.+, C7.1, D1.C, IC2.IN, IC3.IN
- net GND: now also C1.2, C11.1, C12.1, C14.1, C15.1, C16.-, C5.1, D1.A, D2.A, DA1.VSS, DRIVER.10, IC1.GND@1, IC2.VSS, IC3.GND, PROG.5, R15.1, R4.1, R6.1, R7.2; no longer 3,3V.C, 5V.C, 6-30V-2.S, C1.-, C10.2, C11.-, C12.2, C4.1, C5.2, C7.2, DA1.VDD, IC1.GND, IC1.GND@EXP, IC1.GND@M, IC2.ADJ, IC3.ADJ, IC4.GND, R10.1, R2.2, R3.2, RS-485.1, RS-485.5, SV1.16, U1.GND@1, U1.GND@2, U1.GND@3, U1.GND@4, UBS-B.4
- net N$1: now also D3.A, DRIVER.1; no longer IC1.D-, UBS-B.2
- net N$10: now also C3.1, IC1.PB6(XTAL1/TOSC1), Q2.1; no longer IC4.A, R9.1, RS-485.8, S1.S
- net N$11: now also C4.1, IC1.PB7(XTAL2/TOSC2), Q2.2; no longer IC4.B, R10.2, R11.1, RS-485.3
- net N$12: now also +5V.C, R15.2; no longer R11.2, S1.P
- net N$2: now also CAN.C, R7.1; no longer IC1.D+, UBS-B.3
- net N$3: now also CAN.A, IC1.PD5(T1); no longer IC1.!RST, R1.1
- net N$6: now also IC2.!RST, R1.1; no longer 3,3V.A, R4.1
- net SCK: now also IC1.PB5(SCK), IC2.SCK, SC.TP; no longer U1.IO18
Other:
- note added: "BREAK-PWM"
- note added: "CAN-Interface"
- note added: "Controler"
- note added: "DRIVE-PWM"
- note added: "FORW-REL"
- note added: "FTDI-Interface"
- note added: "HORN"
- note added: "LIGHT"
- note added: "Motor V2.1b-s"
- note added: "REVERS-REL"

Commit message: initial
Parts:
- added D4, D5: 5,1V, diode:ZENER-DIODESOD80C
- added P1: (no value), jst-ph:JST-PH2
- added R10, R8: 47K, rcl:R-EU_MELF0102W
- added R11, R9: 10k, rcl:R-EU_MELF0102W
Connections:
- new net A2: D4.C, IC1.PC2(ADC2), R8.1, R9.2
- new net A3: D5.C, IC1.PC3(ADC3), R10.1, R11.2
- new net BATT-1: P1.1, R8.2
- new net BATT-2: P1.2, R10.2
- net GND: now also D4.A, D5.A, R11.1, R9.1
Other:
- note added: "Motor V2.2-s"
- note removed: "Motor V2.1b-s"

Commit message: initial
Other:
- moved on the sheet: C3, C4, C5, C8, CAN, IC1, Q2, R2, R7
