File: V2.x/Servo/LOCO-Servo.brd (EAGLE design)
At the start: 43.2 x 34.3 mm, 48 parts, among them IC1 Atmega 328-P, IC2 MCP2515, IC4 LD117AS12TR, Q1 8MHz, Q2 16MHz, Q8 FDS5680

Commit message: Signed-off-by: Thomas Winkler <thomas.winkler@iggmp.net>
Parts:
- removed D6: BAS40, diode:SOT23
- removed IC4: LD117AS12TR, v-reg:SOT223
- removed Q8: FDS5680, transistor-fet:SO-8
- removed R12, R13: 10k, rcl:MINI_MELF-0102W
- removed S1-2, S3-4: (no value), con-lstb:MA03-2
- removed SWITCH: 22-23-2021, con-molex:22-23-2021
- added CAN: (no value), led:CHIP-LED0603
- added IC3: LM340MP-05, linear:SOT223
- added R14: 10k, rcl:MINI_MELF-0102W
- added SC, SI, SO: PTR1B1,27, testpad:B1,27
- added SDI: (no value), jumper:SJ
- added X2: 2X6-A, con-amp-micro-mate-n-lock:4-794618-2
- moved D3 3.24 mm to (29.8, 15.9), flipped to the top
- moved R10 3.18 mm to (29.8, 24.8), flipped to the top
- moved R9 3.18 mm to (29.8, 21.0), flipped to the top
- moved +5V 3.17 mm to (8.26, 32.4)
- moved R5 2.01 mm to (27.3, 14.6)
- moved D2 2.01 mm to (24.8, 15.9)
- moved R6 2.01 mm to (27.3, 17.8)
- moved R15 1.90 mm to (13.3, 32.4)
- moved R1 0.95 mm to (21.0, 25.1)
- moved D4 0.64 mm to (29.8, 22.9)
- moved R7 0.64 mm to (29.8, 14.6)
- moved R8 0.64 mm to (29.8, 17.8)
- moved D1 0.63 mm to (30.5, 10.2), flipped to the top
- moved R3 0.63 mm to (27.9, 8.26), flipped to the top
- moved R4 0.63 mm to (27.9, 11.4), flipped to the top
Connections:
- removed net A4: D4.C, IC1.27, R10.2, R9.1
- removed net A5: IC1.28
- removed net D6: IC1.10
- removed net D7: IC1.11
- removed net N$8: Q8.4, R12.1, R13.1
- removed net SWITCH1: R12.2
- new net CAN-CS: IC2.18, SDI.2
- new net N$1: CAN.C, R14.1
- net +12V: now also IC3.1; no longer IC4.3
- net A0: now also D1.C, R3.1, R4.2
- net A1: now also D2.C, R5.1, R6.2; no longer D1.C, R3.1, R4.2
- net A2: now also D3.C, R7.1, R8.2; no longer D2.C, R5.1, R6.2
- net A3: now also D4.C, R10.2, R9.1; no longer D3.C, R7.1, R8.2
- net CS: now also SDI.1; no longer IC2.18
- net D9: now also CAN.A
- net GND: now also IC3.4, R14.2, X2.11, X2.12, X2.5, X2.6; no longer D6.1, IC4.1, Q8.1, Q8.2, Q8.3, R13.2, S1-2.5, S1-2.6, S3-4.5, S3-4.6, SWITCH.2
- net RX: now also SV1.2; no longer SV1.3
- net S1: no longer D6.3, Q8.5, Q8.6, Q8.7, Q8.8, SWITCH.1
- net SCK: now also SC.TP
- net SERVO1: now also X2.1; no longer S1-2.1
- net SERVO2: now also X2.2; no longer S1-2.2
- net SERVO3: now also X2.7; no longer S3-4.1
- net SERVO4: now also X2.8; no longer S3-4.2
- net SI: now also SI.TP
- net SO: now also SO.TP
- net TX: now also SV1.3; no longer SV1.2
- net VCC: now also IC3.3, X2.10, X2.3, X2.4, X2.9; no longer IC4.4, S1-2.3, S1-2.4, S3-4.3, S3-4.4
Routing:
- net S1: track 63.0 -> 0.00 mm
- net A0: track 0.00 -> 46.0 mm, vias 0 -> 1
- net GND: track 296.8 -> 261.3 mm, vias 0 -> 1
- net SERVO4: track 50.3 -> 22.6 mm, vias 3 -> 0
- net A4: track 25.5 -> 0.00 mm, vias 3 -> 0
- net SERVO3: track 27.9 -> 51.4 mm, vias 3 -> 1
- net N$6: track 25.7 -> 7.25 mm
- net D9: track 0.00 -> 18.2 mm, vias 0 -> 1
- net A1: track 23.1 -> 7.35 mm
- net SERVO2: track 43.2 -> 30.5 mm, vias 4 -> 2
- net N$8: track 11.5 -> 0.00 mm
- net SERVO1: track 45.7 -> 34.4 mm, vias 2 -> 0
- net A3: track 30.2 -> 19.0 mm, vias 0 -> 2
- net A2: track 10.6 -> 19.7 mm, vias 0 -> 4
- net N$15: track 21.1 -> 30.2 mm, vias 1 -> 3
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Other:
- board text added: "V2.1a-s"
- board text removed: "V2.0"

Commit message: initial
Connections:
- removed net D2: R11.2, SPEED.1
- new net PULSE: IC1.19, R11.2, SPEED.1
Routing:
- net PULSE: track 0.00 -> 15.1 mm, vias 0 -> 3
- net D2: track 6.24 -> 0.00 mm
Changed lines of the file:
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@@
 <autorouter>
 <pass name="Default">
-<param name="RoutingGrid" value="6.25mil"/>
 <param name="AutoGrid" value="0"/>
 <param name="Efforts" value="2"/>
@@
 <wire x1="33.0708" y1="18.8976" x2="33.195" y2="18.765" width="0.1524" layer="1"/>
 <via x="17.3736" y="29.718" extent="1-16" drill="0.35"/>
-<polygon width="0.1524" layer="1">
+<polygon width="0.1524" layer="16">
 <vertex x="0" y="34.29"/>
 <vertex x="43.18" y="34.29"/>
@@
 <vertex x="0" y="0"/>
 </polygon>
-<polygon width="0.1524" layer="16">
+<polygon width="0.1524" layer="1">
 <vertex x="0" y="34.29"/>
 <vertex x="43.18" y="34.29"/>
@@
 <wire x1="15.24" y1="2.5908" x2="15.24" y2="2.54" width="0.1524" layer="16"/>
 </signal>
-<signal name="D2">
-<contactref element="SPEED" pad="1"/>
-<contactref element="R11" pad="2"/>
-<wire x1="30.0228" y1="27.2796" x2="26.3652" y2="23.622" width="0.1524" layer="1"/>
-<wire x1="30.7848" y1="27.2796" x2="30.0228" y2="27.2796" width="0.1524" layer="1"/>
-<wire x1="26.3652" y1="23.622" x2="26.35" y2="23.495" width="0.1524" layer="1"/>
-<wire x1="30.7848" y1="27.2796" x2="30.885" y2="27.43" width="0.1524" layer="1"/>
-</signal>
 <signal name="+12V">
 <contactref element="CAN-1" pad="4"/>
@@
 <wire x1="11.43" y1="30.1752" x2="11.43" y2="30.16" width="0.1524" layer="1"/>
 </signal>
+<signal name="PULSE">
+<contactref element="SPEED" pad="1"/>
+<contactref element="R11" pad="2"/>
+<wire x1="30.0228" y1="27.2796" x2="26.8224" y2="24.0792" width="0.1524" layer="1"/>
+<wire x1="26.8224" y1="24.0792" x2="26.3652" y2="23.622" width="0.1524" layer="1"/>
+<wire x1="30.7848" y1="27.2796" x2="30.0228" y2="27.2796" width="0.1524" layer="1"/>
+<wire x1="26.3652" y1="23.622" x2="26.35" y2="23.495" width="0.1524" layer="1"/>
+<wire x1="30.7848" y1="27.2796" x2="30.885" y2="27.43" width="0.1524" layer="1"/>
+<contactref element="IC1" pad="19"/>
+<wire x1="23.4696" y1="18.7452" x2="22.098" y2="18.7452" width="0.1524" layer="16"/>
+<wire x1="23.9268" y1="18.7452" x2="23.4696" y2="18.7452" width="0.1524" layer="1"/>
+<wire x1="27.1272" y1="21.9456" x2="23.9268" y2="18.7452" width="0.1524" layer="1"/>
+<wire x1="27.1272" y1="23.4696" x2="27.1272" y2="21.9456" width="0.1524" layer="16"/>
+<wire x1="27.2796" y1="23.622" x2="27.1272" y2="23.4696" width="0.1524" layer="16"/>
+<wire x1="26.8224" y1="24.0792" x2="27.2796" y2="23.622" width="0.1524" layer="1"/>
+<wire x1="22.098" y1="18.7452" x2="22.0726" y2="18.6625" width="0.1524" layer="16"/>
+<via x="23.4696" y="18.7452" extent="1-16" drill="0.35"/>
+<via x="27.1272" y="21.9456" extent="1-16" drill="0.35"/>
+<via x="27.2796" y="23.622" extent="1-16" drill="0.35"/>
+</signal>
 </signals>

Commit message: initial
Parts:
- added SO1: PTR1B1,27, testpad:B1,27
- +5V: value (none) -> LED_GREEN; device led:CHIP-LED0603 -> Opto-Electronic:LEDC1608X39N_G
- CAN: value (none) -> STATUS; device led:CHIP-LED0603 -> Opto-Electronic:LEDC1608X39N_B
- D1, D2, D3, D4: value (none) -> 5.1V
- R14: value 10k -> 220R
- moved C4 9.44 mm to (10.8, 20.3), turned to 180 degrees
- moved R2 8.83 mm to (25.1, 15.9), turned to 90 degrees
- moved C8 7.25 mm to (17.5, 9.21), turned to 90 degrees
- moved C2 6.51 mm to (19.7, 6.35)
- moved R15 4.49 mm to (8.89, 31.8), turned to 0 degrees
- moved C1 4.26 mm to (20.3, 9.21), turned to 90 degrees
- moved +5V 4.18 mm to (12.4, 31.8), turned to 0 degrees
- moved C3 3.19 mm to (10.8, 14.0), turned to 180 degrees
- moved SI 1.91 mm to (25.1, 23.5)
- moved SO 1.91 mm to (25.1, 25.1)
- moved SC 1.90 mm to (25.1, 21.9)
- moved CAN 1.42 mm to (8.89, 29.2), turned to 180 degrees
- moved R9 0.71 mm to (30.5, 21.3)
- moved R7 0.71 mm to (30.5, 14.3)
- moved C6 0.71 mm to (12.7, 23.8), turned to 90 degrees
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Connections:
- removed net N$15: C8.2, IC1.29, R2.1
- new net MCU_RESET: C8.2, IC1.29, R2.1, SO1.TP
- new net N$2: CAN.2, IC1.11
- net D9: no longer CAN.A
- net N$1: now also CAN.1; no longer CAN.C
- net N$12: now also +5V.1; no longer +5V.C
- net VCC: now also +5V.2; no longer +5V.A
Routing:
- net GND: track 261.3 -> 205.7 mm, vias 1 -> 3
- net MCU_RESET: track 0.00 -> 31.9 mm, vias 0 -> 2
- net N$15: track 30.2 -> 0.00 mm, vias 3 -> 0
- net SERVO1: track 34.4 -> 56.4 mm, vias 0 -> 1
- net A0: track 46.0 -> 27.8 mm
- net D9: track 18.2 -> 0.00 mm, vias 1 -> 0
- net N$2: track 0.00 -> 14.2 mm, vias 0 -> 1
- net VCC: track 155.5 -> 142.6 mm
- net +12V: track 39.5 -> 50.5 mm
- net SERVO3: track 51.4 -> 44.4 mm, vias 1 -> 2
- net CAN-CS: track 8.28 -> 3.20 mm, vias 2 -> 0
- net A2: track 19.7 -> 15.0 mm, vias 4 -> 2
- net N$6: track 7.25 -> 12.0 mm
- net PULSE: track 15.1 -> 19.4 mm, vias 3 -> 0
- net SCK: track 12.5 -> 8.70 mm, vias 2 -> 1
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Other:
- board text added: "V2.1b-s"
