File: V2.x/Servo/LOCO-Servo.sch (EAGLE design)
At the start: 48 parts, among them IC1 Atmega 328-P, IC2 MCP2515, IC4 LD117AS12TR, Q1 8MHz, Q2 16MHz, Q8 FDS5680

Commit message: Signed-off-by: Thomas Winkler <thomas.winkler@iggmp.net>
Parts:
- removed D6: BAS40, diode:BAS40
- removed IC4: LD117AS12TR, v-reg:LD117AS12TR
- removed Q8: FDS5680, transistor-fet:FDS5680
- removed R12, R13: 10k, rcl:R-EU_MELF0102W
- removed S1-2, S3-4: (no value), con-lstb:MA03-2
- removed SWITCH: 22-23-2021, con-molex:22-23-2021
- added CAN: (no value), led:LEDCHIP-LED0603
- added IC3: LM340MP-05, linear:LM340MP-05
- added R14: 10k, rcl:R-EU_MELF0102W
- added SC, SI, SO: PTR1B1,27, testpad:PTR1B1,27
- added SDI: (no value), jumper:SJ
- added X2: 2X6-A, con-amp-micro-mate-n-lock:2X6-A
Connections:
- removed net A4: D4.C, IC1.PC4(ADC4/SDA), R10.2, R9.1
- removed net A5: IC1.PC5(ADC5/SCL)
- removed net D6: IC1.PD6(AIN0)
- removed net D7: IC1.PD7(AIN1)
- removed net N$8: Q8.G, R12.1, R13.1
- removed net SWITCH1: R12.2
- new net CAN-CS: IC2.!CS, SDI.2
- new net N$1: CAN.C, R14.1
- net +12V: now also IC3.VI; no longer IC4.IN
- net A0: now also D1.C, R3.1, R4.2
- net A1: now also D2.C, R5.1, R6.2; no longer D1.C, R3.1, R4.2
- net A2: now also D3.C, R7.1, R8.2; no longer D2.C, R5.1, R6.2
- net A3: now also D4.C, R10.2, R9.1; no longer D3.C, R7.1, R8.2
- net CS: now also SDI.1; no longer IC2.!CS
- net D9: now also CAN.A
- net GND: now also IC3.GND, R14.2, X2.11.S, X2.12.S, X2.5.S, X2.6.S; no longer D6.A, IC4.ADJ, Q8.S, R13.2, S1-2.5, S1-2.6, S3-4.5, S3-4.6, SWITCH-2.S
- net RX: now also SV1.2; no longer SV1.3
- net S1: no longer D6.C, Q8.D, SWITCH-1.S
- net SCK: now also SC.TP
- net SERVO1: now also X2.1.S; no longer S1-2.1
- net SERVO2: now also X2.2.S; no longer S1-2.2
- net SERVO3: now also X2.7.S; no longer S3-4.1
- net SERVO4: now also X2.8.S; no longer S3-4.2
- net SI: now also SI.TP
- net SO: now also SO.TP
- net TX: now also SV1.3; no longer SV1.2
- net VCC: now also IC3.VO, X2.10.S, X2.3.S, X2.4.S, X2.9.S; no longer IC4.OUT, S1-2.3, S1-2.4, S3-4.3, S3-4.4
Other:
- note added: "LOCO-Servo V2.1a-s"
- moved on the sheet: +5V, C1, C11, C12, C13, C14, C15, C16, C2, C6, CAN-1, CAN-2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

Commit message: initial
Connections:
- removed net D2: R11.2, SPEED.1
- new net PULSE: IC1.ADC6, R11.2, SPEED.1
Changed lines of the file:
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@@
-</segment>
-</net>
-<net name="D2" class="0">
-<segment>
-<pinref part="SPEED" gate="G$1" pin="1"/>
-<wire x1="0" y1="-91.44" x2="-12.7" y2="-91.44" width="0.1524" layer="91" grouprefs="SPEEDO"/>
-<pinref part="R11" gate="G$1" pin="2"/>
-<wire x1="-12.7" y1="-91.44" x2="-22.86" y2="-91.44" width="0.1524" layer="91" grouprefs="SPEEDO"/>
-<wire x1="-12.7" y1="-88.9" x2="-12.7" y2="-91.44" width="0.1524" layer="91" grouprefs="SPEEDO"/>
-<junction x="-12.7" y="-91.44" grouprefs="SPEEDO"/>
-<label x="-20.32" y="-91.44" size="1.778" layer="95" grouprefs="SPEEDO"/>
 </segment>
 </net>
@@
 </segment>
 </net>
+<net name="PULSE" class="0">
+<segment>
+<pinref part="SPEED" gate="G$1" pin="1"/>
+<wire x1="0" y1="-91.44" x2="-12.7" y2="-91.44" width="0.1524" layer="91" grouprefs="SPEEDO"/>
+<pinref part="R11" gate="G$1" pin="2"/>
+<wire x1="-12.7" y1="-91.44" x2="-22.86" y2="-91.44" width="0.1524" layer="91" grouprefs="SPEEDO"/>
+<wire x1="-12.7" y1="-88.9" x2="-12.7" y2="-91.44" width="0.1524" layer="91" grouprefs="SPEEDO"/>
+<junction x="-12.7" y="-91.44" grouprefs="SPEEDO"/>
+<label x="-20.32" y="-91.44" size="1.778" layer="95" grouprefs="SPEEDO"/>
+</segment>
+<segment>
+<pinref part="IC1" gate="G$1" pin="ADC6"/>
+<wire x1="55.88" y1="58.42" x2="71.12" y2="58.42" width="0.1524" layer="91"/>
+<label x="66.04" y="58.42" size="1.778" layer="95"/>
+</segment>
+</net>

Commit message: initial
Parts:
- added SO1: PTR1B1,27, testpad:PTR1B1,27
- +5V: value (none) -> LED_GREEN; device led:LEDCHIP-LED0603 -> Opto-Electronic:LED_CHIP_GREEN-1608
- CAN: value (none) -> STATUS; device led:LEDCHIP-LED0603 -> Opto-Electronic:LED_CHIP_BLUE-1608
- D1, D2, D3, D4: value (none) -> 5.1V
- R14: value 10k -> 220R
Connections:
- removed net N$15: C8.2, IC1.PC6(/RESET), R2.1
- new net MCU_RESET: C8.2, IC1.PC6(/RESET), R2.1, SO1.TP
- new net N$2: CAN.A, IC1.PD7(AIN1)
- net D9: no longer CAN.A
- net GND: now also IC1.GND@2
- net VCC: now also IC1.VCC@2
Other:
- note added: "LOCO-Servo V2.1b-s"
- note removed: "LOCO-Servo V2.1a-s"
- moved on the sheet: SC, SI, SO
