File: V2.x/Split/Split.brd (EAGLE design)
At the start: 30.5 x 17.8 mm, 6 parts, among them J1 3-794618-4, J2 3-794618-4, J3 3-794618-4, X2 2X1-A

Commit message: initial
Parts:
- moved C1 0.48 mm to (15.4, 2.22)
- renumbered X2 to PWR
Connections:
- net +12V: now also D1.C; no longer PWR.2
- net GND: now also PWR.2; no longer D1.C
Routing:
- net GND: track 24.2 -> 34.3 mm
- net +12V: track 39.5 -> 45.1 mm
- net N$5: track 28.0 -> 29.5 mm
- added copper zone on layer 1, net +12V
- removed copper zone on layer 1, net GND
