File: V2.x/Universal/Universal.brd (EAGLE design)
At the start: 34.3 x 34.3 mm, 28 parts, among them IC1 Atmega 328-P, IC2 MCP2515, IC4 LD117AS12TR, Q1 8MHz, Q2 16MHz

Commit message: Signed-off-by: Thomas Winkler <thomas.winkler@iggmp.net>
Parts:
- removed BUS: (no value), con-lstb:MA09-2
- removed IC4: LD117AS12TR, v-reg:SOT223
- removed PWR: 22-23-2021, con-molex:22-23-2021
- removed SV1: (no value), con-lstb:MA05-1
- added BUS1: (no value), con-lstb:MA09-1
- added BUS2A, ICP: (no value), con-lstb:MA05-1
- added BUS2B: (no value), con-lstb:MA04-1
- added CS: (no value), jumper:SJ
- added D2: (no value), diode:DO214AA
- added IC3: LM340MP-05, linear:SOT223
- added SC, SI, SO: PTR1B1,27, testpad:B1,27
- R15: value 10k -> 220R
- moved C4 27.7 mm to (27.9, 7.62), flipped to the top
- moved Q2 20.5 mm to (27.0, 14.3), turned to 270 degrees
- moved C3 16.3 mm to (27.0, 20.6), flipped to the top, turned to 0 degrees
- moved DA1 13.5 mm to (6.03, 17.1)
- moved C2 12.9 mm to (12.7, 7.62), flipped to the top, turned to 90 degrees
- moved C1 11.8 mm to (25.7, 7.62), flipped to the top, turned to 90 degrees
- moved Q1 9.23 mm to (19.4, 7.62), turned to 180 degrees
- moved C5 8.67 mm to (11.4, 13.7), flipped to the bottom, turned to 90 degrees
- moved R15 8.14 mm to (12.4, 24.8), turned to 90 degrees
- moved C11 7.36 mm to (12.4, 21.9), turned to 0 degrees
- moved C15 7.36 mm to (25.7, 28.3), flipped to the top
- moved C6 7.36 mm to (12.4, 16.8), flipped to the top
- moved C16 6.79 mm to (27.9, 24.8), flipped to the top
- moved C12 5.48 mm to (12.4, 20.3), turned to 0 degrees
- moved +5V 4.86 mm to (12.4, 27.6), turned to 180 degrees
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Connections:
- removed net 12V-PWR: BUS.17, PWR.1
- new net CAN-CS: CS.2, IC2.18
- new net N$2: BUS2A.1, D2.A
- net +12V: now also D2.C, IC3.1; no longer IC4.3
- net A0: now also BUS2B.2; no longer BUS.13
- net A1: now also BUS2B.1; no longer BUS.11
- net A2: now also BUS2A.5; no longer BUS.9
- net A3: now also BUS2A.4; no longer BUS.7
- net A4: now also BUS2A.3; no longer BUS.5
- net A5: now also BUS2A.2; no longer BUS.3
- net CS: now also CS.1; no longer IC2.18
- net D2: now also BUS1.2; no longer BUS.2
- net D3: now also BUS1.3; no longer BUS.4
- net D4: now also BUS1.4; no longer BUS.6
- net D5: now also BUS1.5; no longer BUS.8
- net D6: now also BUS1.6; no longer BUS.10
- net D7: now also BUS1.7; no longer BUS.12
- net D8: now also BUS1.8; no longer BUS.14
- net D9: now also BUS2B.3; no longer BUS.15
- net DTR: now also ICP.1; no longer SV1.1
- net GND: now also BUS1.9, BUS2B.4, IC3.4, ICP.5; no longer BUS.16, BUS.18, IC4.1, PWR.2, SV1.5
- net RX: now also ICP.2; no longer SV1.3
- net SCK: now also SC.TP
- net SI: now also SI.TP
- net SO: now also SO.TP
- net TX: now also ICP.3; no longer SV1.2
- net VCC: now also BUS1.1, IC3.3, ICP.4; no longer BUS.1, IC4.4, SV1.4
Routing:
- net VCC: track 143.7 -> 93.3 mm, vias 9 -> 7
- net D2: track 20.4 -> 68.2 mm, vias 2 -> 6
- net SCK: track 4.92 -> 43.9 mm
- net A2: track 47.3 -> 12.4 mm, vias 7 -> 0
- net 12V-PWR: track 29.1 -> 0.00 mm, vias 2 -> 0
- net N$15: track 37.9 -> 14.4 mm, vias 3 -> 1
- net CAN-CS: track 0.00 -> 21.2 mm, vias 0 -> 1
- net A5: track 31.4 -> 15.0 mm, vias 2 -> 0
- net A4: track 27.8 -> 13.9 mm, vias 1 -> 0
- net D5: track 24.4 -> 10.8 mm, vias 2 -> 0
- net D9: track 15.8 -> 29.0 mm
- net D8: track 25.2 -> 13.3 mm, vias 1 -> 0
- net +12V: track 38.5 -> 50.0 mm
- net A1: track 24.6 -> 13.5 mm, vias 1 -> 0
- net SO: track 4.91 -> 15.5 mm
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Other:
- board text added: "LOCO"
- board text added: "Universal"
- board text added: "V2.1-s"
- board text removed: "LOCO-Universal"
- board text removed: "V2.0"

Commit message: initial
Parts:
- added CAN: Status, led:SML0603
- added R3: 220R, rcl:MINI_MELF-0102W
- added SO1: PTR1B1,27, testpad:B1,27
- moved C2 0.99 mm to (13.0, 6.67)
- moved C8 0.64 mm to (23.8, 15.2)
- moved C5 0.32 mm to (11.4, 14.0)
Connections:
- removed net N$15: C8.2, IC1.29, R2.1
- new net MCU_RESET: C8.2, IC1.29, R2.1, SO1.TP
- new net N$1: IC1.19, R3.1
- new net N$3: CAN.A, R3.2
- net GND: now also CAN.C
Routing:
- net D2: track 68.2 -> 25.1 mm, vias 6 -> 0
- net MCU_RESET: track 0.00 -> 32.9 mm, vias 0 -> 2
- net SCK: track 43.9 -> 16.8 mm
- net SI: track 12.9 -> 33.5 mm
- net GND: track 142.3 -> 159.9 mm, vias 1 -> 0
- net VCC: track 93.3 -> 108.0 mm, vias 7 -> 4
- net N$15: track 14.4 -> 0.00 mm, vias 1 -> 0
- net D9: track 29.0 -> 38.7 mm, vias 2 -> 0
- net SO: track 15.5 -> 10.2 mm
- net N$6: track 10.8 -> 15.6 mm, vias 1 -> 3
- net N$1: track 0.00 -> 4.59 mm
- net CAN-CS: track 21.2 -> 17.2 mm
- net N$3: track 0.00 -> 3.95 mm, vias 0 -> 1
- net CAN-H: track 30.1 -> 28.1 mm, vias 0 -> 2
- net CS: track 9.79 -> 8.63 mm, vias 2 -> 0
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Other:
- board text added: "V2.2-s"
- board text removed: "V2.1-s"
