File: V2.x/Universal/Universal.sch (EAGLE design)
At the start: 28 parts, among them IC1 Atmega 328-P, IC2 MCP2515, IC4 LD117AS12TR, Q1 8MHz, Q2 16MHz

Commit message: Signed-off-by: Thomas Winkler <thomas.winkler@iggmp.net>
Parts:
- removed BUS: (no value), con-lstb:MA09-2
- removed IC4: LD117AS12TR, v-reg:LD117AS12TR
- removed PWR: 22-23-2021, con-molex:22-23-2021
- removed SV1: (no value), con-lstb:MA05-1
- added BUS1: (no value), con-lstb:MA09-1
- added BUS2A, ICP: (no value), con-lstb:MA05-1
- added BUS2B: (no value), con-lstb:MA04-1
- added CS: (no value), jumper:SJ
- added D2: (no value), diode:DIODE-DO214AA
- added IC3: LM340MP-05, linear:LM340MP-05
- added SC, SI, SO: PTR1B1,27, testpad:PTR1B1,27
- R15: value 10k -> 220R
Connections:
- removed net 12V-PWR: BUS.17, PWR-1.S
- new net CAN-CS: CS.2, IC2.!CS
- new net N$2: BUS2A.1, D2.A
- net +12V: now also D2.C, IC3.VI; no longer IC4.IN
- net A0: now also BUS2B.2; no longer BUS.13
- net A1: now also BUS2B.1; no longer BUS.11
- net A2: now also BUS2A.5; no longer BUS.9
- net A3: now also BUS2A.4; no longer BUS.7
- net A4: now also BUS2A.3; no longer BUS.5
- net A5: now also BUS2A.2; no longer BUS.3
- net CS: now also CS.1; no longer IC2.!CS
- net D2: now also BUS1.2; no longer BUS.2
- net D3: now also BUS1.3; no longer BUS.4
- net D4: now also BUS1.4; no longer BUS.6
- net D5: now also BUS1.5; no longer BUS.8
- net D6: now also BUS1.6; no longer BUS.10
- net D7: now also BUS1.7; no longer BUS.12
- net D8: now also BUS1.8; no longer BUS.14
- net D9: now also BUS2B.3; no longer BUS.15
- net DTR: now also ICP.1; no longer SV1.1
- net GND: now also BUS1.9, BUS2B.4, IC3.GND, ICP.5; no longer BUS.16, BUS.18, IC4.ADJ, PWR-2.S, SV1.5
- net RX: now also ICP.2; no longer SV1.3
- net SCK: now also SC.TP
- net SI: now also SI.TP
- net SO: now also SO.TP
- net TX: now also ICP.3; no longer SV1.2
- net VCC: now also BUS1.1, IC3.VO, ICP.4; no longer BUS.1, IC4.OUT, SV1.4
Other:
- note added: "FTDI-Interface"
- note added: "In 2.1 version"
- note added: "LOCO-Universal 2.1-s"
- note added: "RX and TX are swapped"
- note removed: "IFTDI-Interface"
- moved on the sheet: +5V, C1, C11, C12, C13, C14, C15, C16, C2, C6, CAN-1, CAN-2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

Commit message: initial
Parts:
- added CAN: Status, led:LEDSML0603
- added R3: 220R, rcl:R-EU_MELF0102W
- added SO1: PTR1B1,27, testpad:PTR1B1,27
Connections:
- removed net N$15: C8.2, IC1.PC6(/RESET), R2.1
- new net MCU_RESET: C8.2, IC1.PC6(/RESET), R2.1, SO1.TP
- new net N$1: IC1.ADC6, R3.1
- new net N$3: CAN.A, R3.2
- net GND: now also CAN.C
Other:
- note added: "LOCO-Universal 2.2-s"
- note added: "On the motor driver, the polarity of D2 has to be swapped."
- note removed: "LOCO-Universal 2.1-s"
- moved on the sheet: +5V, BUS1, BUS2A, BUS2B, C1, C11, C12, C13, C14, C15, C16, C2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
