File: V2.x/Universal Control Adapter/LOCO-Univ-Control-Adapter.brd (EAGLE design)
At the start: 62.9 x 34.3 mm, 34 parts, among them IC5 LM340MP-05, Q8 FDS5680

Commit message: initial
Connections:
- removed net N$2: BUS2A.1
- net +12V: now also BUS2A.1
Routing:
- net VCC: track 180.1 -> 131.8 mm, vias 2 -> 0
- net +12V: track 16.1 -> 37.3 mm, vias 0 -> 1
- net A1: track 36.9 -> 51.7 mm
- net SUPL: track 41.3 -> 31.2 mm, vias 0 -> 1
- net D5: track 46.8 -> 55.3 mm, vias 1 -> 0
- net GREEN: track 14.4 -> 21.7 mm
- net A0: track 37.8 -> 30.6 mm
- net INSTR-LIGHT: track 24.2 -> 17.3 mm
- net RED: track 14.8 -> 21.4 mm
- net D8: track 53.1 -> 59.3 mm, vias 1 -> 0
- net GND: track 211.7 -> 216.5 mm
- net D9: track 58.0 -> 61.5 mm
- net A2: track 41.9 -> 43.4 mm, vias 1 -> 3
- net A3: track 37.3 -> 38.8 mm, vias 0 -> 1
- net A4: track 49.1 -> 50.2 mm
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