File: V2.x/Universal WiFi/Universal-WIFI.brd (EAGLE design)
At the start: 34.3 x 34.3 mm, 28 parts, among them IC1 LM340MP-05, IC2 LD117AS33TR, U1 ESP-WROOM-32ESP-WROOM-32-ANT

Commit message: initial
Parts:
- added R5: 10k, rcl:R0805
- moved COM 1.59 mm to (32.1, 27.9), turned to 180 degrees
Connections:
- new net EN: PROG.1, R5.1, U1.3
- net +3V3: now also R5.2; no longer U1.3
- net IO0: no longer PROG.1
Routing:
- net IO32: track 78.9 -> 10.5 mm, vias 9 -> 0
- net EN: track 0.00 -> 38.8 mm, vias 0 -> 2
- net GND: track 165.2 -> 184.8 mm, vias 2 -> 1
- net IO0: track 13.2 -> 0.00 mm, vias 1 -> 0
- net +3V3: track 79.5 -> 91.1 mm, vias 1 -> 3
- net IO14: track 38.0 -> 46.2 mm, vias 0 -> 2
- net IO15: track 30.9 -> 24.8 mm, vias 0 -> 1
- net +5V: track 32.1 -> 37.3 mm, vias 3 -> 2
- net IO13: track 35.4 -> 30.7 mm, vias 2 -> 1
- net CAN-TX: track 43.5 -> 38.9 mm, vias 2 -> 4
- net RXD0: track 4.24 -> 7.88 mm, vias 0 -> 1
- net IO34: track 16.3 -> 13.0 mm, vias 1 -> 0
- net N$2: track 2.98 -> 5.45 mm
- net N$8: track 31.9 -> 34.3 mm
- net +12V: track 56.3 -> 53.9 mm
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- removed copper zone on layer 1, net GND
- removed copper zone on layer 16, net GND
Other:
- board text added: "V2.1b"
- board text removed: "V2.1a"

Commit message: initial
Parts:
- removed COM: (no value), led:CHIPLED_0603
- removed PROG: (no value), con-lstb:MA05-1
- added SV1: (no value), con-lstb:MA06-1
- added WIFI: LED_BLUE, Opto-Electronic:LEDC1608X39N_B
- 3,3V: value (none) -> LED_RED; device led:CHIPLED_0603 -> Opto-Electronic:LEDC1608X39N_R
- 5V: value (none) -> LED_GREEN; device led:CHIPLED_0603 -> Opto-Electronic:LEDC1608X39N_G
- moved R5 0.71 mm to (28.9, 27.9)
Connections:
- net +3V3: now also SV1.5; no longer PROG.4
- net EN: now also SV1.2; no longer PROG.1
- net GND: now also 3,3V.1, 5V.1, SV1.6, WIFI.1; no longer 3,3V.C, 5V.C, COM.C, PROG.5
- net IO0: now also SV1.1
- net N$13: now also 5V.2; no longer 5V.A
- net N$3: now also WIFI.2; no longer COM.A
- net N$6: now also 3,3V.2; no longer 3,3V.A
- net RXD0: now also SV1.3; no longer PROG.2
- net TXD0: now also SV1.4; no longer PROG.3
Routing:
- net CAN-TX: track 38.9 -> 59.4 mm, vias 4 -> 2
- net IO0: track 0.00 -> 13.6 mm, vias 0 -> 1
- net GND: track 184.8 -> 171.6 mm, vias 1 -> 3
- net +3V3: track 91.1 -> 103.4 mm, vias 3 -> 2
- net IO14: track 46.2 -> 37.9 mm, vias 2 -> 0
- net IO13: track 30.7 -> 38.3 mm
- net IO15: track 24.8 -> 30.8 mm, vias 1 -> 0
- net EN: track 38.8 -> 33.2 mm, vias 2 -> 6
- net CAN-RX: track 27.1 -> 21.8 mm, vias 3 -> 2
- net RXD0: track 7.88 -> 3.37 mm, vias 1 -> 0
- net +5V: track 37.3 -> 40.4 mm
- net N$2: track 5.45 -> 2.98 mm
- net IO12: track 41.4 -> 39.1 mm
- net IO35: track 11.8 -> 13.2 mm
- net N$6: track 2.76 -> 3.81 mm
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- added copper zone on layer 1, net GND
- added copper zone on layer 16, net GND
