File: V2.x/Universal WiFi/Universal-WIFI.sch (EAGLE design)
At the start: 48 parts, among them IC1 Atmega 328-P, IC2 MCP2515, IC4 LD117AS12TR, IC5 ACS750LCA-050, Q1 8MHz, Q2 16MHz, Q8 FDS5680, X1 06-JST-B6B-XH-A

Commit message: Signed-off-by: Thomas Winkler <thomas.winkler@iggmp.net>
Parts:
- removed +5V: (no value), led:LEDCHIP-LED0603
- removed C+BOT, C+TOP, C-BOT1, C-TOP1, M+-BOT, M+-TOP, M--BOT1, M--TOP1: PAD 5.5, holes:MOUNT-PAD-ROUND5.5
- removed C14, C17: 1n, rcl:C-EUC0402K
- removed C15: 100n, rcl:C-EUC0402K
- removed C16: 16uF, rcl:CPOL-EUA/3216-18W
- removed C2, C3, C4: 22p, rcl:C-EUC0402K
- removed D2: (no value), diode:ZENER-DIODESOD80C
- removed IC4: LD117AS12TR, v-reg:LD117AS12TR
- removed IC5: ACS750LCA-050, allegro:ACS750LCA-050
- removed Q1: 8MHz, crystal:CRYSTALHC49S
- removed Q2: 16MHz, crystal:CRYSTALHC49S
- removed Q8: FDS5680, transistor-fet:FDS5680
- removed R15, R6, R7, R8: 10k, rcl:R-EU_R0805
- removed R5: 220K, rcl:R-EU_R0805
- removed SV1: (no value), con-lstb:MA05-1
- removed U$1: FRA2C-2, relais_auto:FRA2C-2
- removed X1: 06-JST-B6B-XH-A, bt_con-jst-xh:06-JST-B6B-XH-A
- added 3,3V, 5V, COM: (no value), led:LEDCHIPLED_0603
- added BUS1: (no value), con-lstb:MA09-1
- added BUS2A, PROG: (no value), con-lstb:MA05-1
- added BUS2B: (no value), con-lstb:MA04-1
- added C10: 100n, rcl:C-EUC0402
- added R12: 220R, rcl:R-EU_R0805
- added U1: ESP-WROOM-32ESP-WROOM-32-ANT, esp32:ESP-WROOM-32ESP-WROOM-32-ANT
- C1: value 22p -> 47uF; device rcl:C-EUC0402K -> rcl:CPOL-EUB/3528-21R
- C11: value 100n -> 47uF; device rcl:C-EUC0402K -> rcl:CPOL-EUB/3528-21R
- C12: value 1n -> 100n; device rcl:C-EUC0402K -> rcl:C-EUC0402
- C13: value 16uF -> 47uF; device rcl:CPOL-EUA/3216-18W -> rcl:CPOL-EUB/3528-21R
- C5: value 100n -> 1uF; device rcl:C-EUC0402K -> rcl:C-EUC0402
- C6, C7, C8: device rcl:C-EUC0402K -> rcl:C-EUC0402
- D1: device diode:ZENER-DIODESOD80C -> diode:DIODE-DO-214AC
- DA1: value TJA1050 -> MCP2551
- IC1: value Atmega 328-P -> LM340MP-05; device atmel:MEGA8-AI -> linear:LM340MP-05
- IC2: value MCP2515 -> LD117AS33TR; device mcp2514:MCP2515 -> v-reg:LD117AS33TR
- R1, R4: value 10k -> 220R
- R2: value 10k -> 5K
- R3: value 220K -> 10K
Connections:
- net CAN-H renamed N$8
- net CAN-L renamed N$9
- removed net A0: C17.2, IC1.PC0(ADC0), IC5.VOUT
- removed net A1: D1.C, IC1.PC1(ADC1), R3.1, R4.2
- removed net A2: D2.C, IC1.PC2(ADC2), R5.1, R6.2
- removed net A3: IC1.PC3(ADC3)
- removed net A4: IC1.PC4(ADC4/SDA)
- removed net A5: IC1.PC5(ADC5/SCL)
- removed net C-: C+BOT.MOUNT, C+TOP.MOUNT, U$1G$2.NO
- removed net C-1: IC5.IP+, U$1G$2.COM
- removed net CAN-OCC1: C1.1, IC2.OSC1, Q1.1
- removed net CAN-OCC2: C2.1, IC2.OSC2, Q1.2
- removed net CS: IC1.PB2(SS/OC1B), IC2.!CS
- removed net D2: IC1.PD2(INT0), X1-5.1
- removed net D3: IC1.PD3(INT1), X1-6.1
- removed net D4: IC1.PD4(XCK/T0), R7.1
- removed net D5: IC1.PD5(T1)
- removed net D6: IC1.PD6(AIN0), X1-2.1
- removed net D7: IC1.PD7(AIN1), X1-3.1
- removed net D8: IC1.PB0(ICP), X1-4.1
- removed net D9: IC1.PB1(OC1A), X1-1.1
- removed net DTR: C8.1, SV1.1
- removed net M+: IC5.IP-, M+-BOT.MOUNT, M+-TOP.MOUNT, R3.2
- removed net M-: C-BOT1.MOUNT, C-TOP1.MOUNT, M--BOT1.MOUNT, M--TOP1.MOUNT, R5.2
- removed net N$10: C3.1, IC1.PB6(XTAL1/TOSC1), Q2.1
- removed net N$11: C4.1, IC1.PB7(XTAL2/TOSC2), Q2.2
- removed net N$12: +5V.C, R15.2
- removed net N$15: C8.2, IC1.PC6(/RESET), R2.1
- removed net RX: IC1.PD1(TXD), SV1.3
- removed net RXCAN: DA1.RXD, IC2.RXCAN
- removed net SCK: IC1.PB5(SCK), IC2.SCK
- removed net SI: IC1.PB4(MISO), IC2.SO
- removed net SO: IC1.PB3(MOSI/OC2), IC2.SI
- removed net TX: IC1.PD0(RXD), SV1.2
- removed net TXCAN: DA1.TXD, IC2.TXCAN
- removed net VCC: +5V.A, C14.2, C15.2, C16.+, C5.2, C6.1, C7.2, DA1.VDD, IC1.AVCC, IC1.VCC@1, IC2.VDD, IC4.OUT, IC5.VCC, R1.2, R2.2, SV1.4
- new net +3V3: BUS1.1, C10.1, C11.+, C5.1, C6.1, IC2.OUT, PROG.4, R4.2, U1.3V3, U1.EN
- new net +5V: C12.1, C13.+, C8.1, DA1.VDD, IC1.VO, IC2.IN, R12.2
- new net CAN-RX: R2.2, R3.2, U1.SD3, U1.SENSOR_VP
- new net CAN-TX: DA1.TXD, U1.SD2, U1.SENSOR_VN
- new net IO0: BUS2A.3, PROG.1, U1.IO0
- new net IO12: BUS2B.2, U1.IO12
- new net IO13: BUS2B.1, U1.IO13
- new net IO14: BUS2B.3, U1.IO14
- new net IO15: BUS2A.5, U1.IO15
- new net IO2: BUS2A.4, U1.IO2
- new net IO25: BUS1.4, U1.IO25
- new net IO26: BUS1.3, U1.IO26
- new net IO27: BUS1.2, U1.IO27
- new net IO32: BUS1.6, U1.IO32
- new net IO33: BUS1.5, U1.IO33
- new net IO34: BUS1.8, U1.IO34
- new net IO35: BUS1.7, U1.IO35
- new net IO4: BUS2A.2, U1.IO4
- new net MCP-RX: DA1.RXD, R2.1
- new net N$13: 5V.A, R12.1
- new net N$3: COM.A, R1.1
- new net RXD0: PROG.2, U1.RXD0
- new net TXD0: PROG.3, U1.TXD0
- net +12V: now also C1.+, C7.1, D1.C, IC1.VI; no longer C11.2, C12.2, C13.+, IC4.IN, U$1G$1.C2
- net GND: now also 3,3V.C, 5V.C, BUS1.9, BUS2B.4, C1.-, C10.2, C11.-, C12.2, C5.2, C7.2, C8.2, COM.C, IC1.GND, IC2.ADJ, PROG.5, R3.1, U1.GND@1, U1.GND@2, U1.GND@3, U1.GND@4; no longer C1.2, C11.1, C12.1, C14.1, C15.1, C16.-, C17.1, C2.2, C3.2, C4.2, C5.1, C7.1, D1.A, D2.A, IC1.GND@1, IC2.VSS, IC4.ADJ, IC5.GND, Q8.S, R15.1, R4.1, R6.1, R8.1, SV1.5
- net N$1: now also BUS2A.1, D1.A; no longer Q8.D, U$1G$1.C1
- net N$2: now also R1.2, U1.IO16; no longer Q8.G, R7.2, R8.2
- net N$6: now also 3,3V.A, R4.1; no longer IC2.!RST, R1.1
Other:
- note added: "WIFI-Controller V2.1a"
- note removed: "BREAK-PWM"
- note removed: "CAN-Interface"
- note removed: "Controler"
- note removed: "DRIVE-PWM"
- note removed: "FORW-REL"
- note removed: "HORN"
- note removed: "IFTDI-Interface"
- note removed: "LIGHT"
- note removed: "REVERS-REL"

Commit message: initial
Parts:
- added R5: 10k, rcl:R-EU_R0805
Connections:
- new net EN: PROG.1, R5.1, U1.EN
- net +3V3: now also R5.2; no longer U1.EN
- net IO0: no longer PROG.1
Other:
- note added: "WIFI-Controller V2.1b"
- note removed: "WIFI-Controller V2.1a"
Changed lines of the file:
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@@
 <part name="R3" library="rcl" library_urn="urn:adsk.eagle:library:334" deviceset="R-EU_" device="R0805" package3d_urn="urn:adsk.eagle:package:23553/2" value="10K"/>
 <part name="GND6" library="supply1" library_urn="urn:adsk.eagle:library:371" deviceset="GND" device=""/>
+<part name="R5" library="rcl" library_urn="urn:adsk.eagle:library:334" deviceset="R-EU_" device="R0805" package3d_urn="urn:adsk.eagle:package:23553/2" value="10k"/>
 </parts>
 <sheets>
 <sheet>
 <plain>
-<text x="-215.9" y="162.56" size="1.778" layer="95">WIFI-Controller V2.1a</text>
+<text x="-215.9" y="162.56" size="1.778" layer="95">WIFI-Controller V2.1b</text>
 </plain>
 <instances>
@@
 <instance part="GND6" gate="1" x="-208.28" y="109.22" smashed="yes" rot="MR0" grouprefs="CAN-INTERFACE">
 <attribute name="VALUE" x="-205.74" y="106.68" size="1.778" layer="96" rot="MR0"/>
+</instance>
+<instance part="R5" gate="G$1" x="-71.12" y="147.32" smashed="yes" rot="R180">
+<attribute name="NAME" x="-67.31" y="145.8214" size="1.778" layer="95" rot="R180"/>
+<attribute name="VALUE" x="-67.31" y="150.622" size="1.778" layer="96" rot="R180"/>
 </instance>
 </instances>
@@
 <pinref part="+3V1" gate="G$1" pin="+3V3"/>
 <pinref part="U1" gate="G$1" pin="3V3"/>
-<wire x1="-86.36" y1="149.86" x2="-86.36" y2="144.78" width="0.1524" layer="91" grouprefs="MCU"/>
+<wire x1="-86.36" y1="149.86" x2="-86.36" y2="147.32" width="0.1524" layer="91" grouprefs="MCU"/>
+<wire x1="-86.36" y1="147.32" x2="-86.36" y2="144.78" width="0.1524" layer="91" grouprefs="MCU"/>
 <wire x1="-86.36" y1="144.78" x2="-78.74" y2="144.78" width="0.1524" layer="91" grouprefs="MCU"/>
 <pinref part="C6" gate="G$1" pin="1"/>
@@
 <junction x="-86.36" y="144.78" grouprefs="MCU"/>
 <pinref part="C5" gate="G$1" pin="1"/>
-<pinref part="U1" gate="G$1" pin="EN"/>
-<wire x1="-78.74" y1="137.16" x2="-78.74" y2="142.24" width="0.1524" layer="91" grouprefs="MCU"/>
-<wire x1="-78.74" y1="142.24" x2="-45.72" y2="142.24" width="0.1524" layer="91" grouprefs="MCU"/>
-<wire x1="-78.74" y1="142.24" x2="-78.74" y2="144.78" width="0.1524" layer="91"/>
-<junction x="-78.74" y="142.24"/>
+<wire x1="-78.74" y1="137.16" x2="-78.74" y2="144.78" width="0.1524" layer="91" grouprefs="MCU"/>
 <junction x="-78.74" y="144.78"/>
+<pinref part="R5" gate="G$1" pin="2"/>
+<wire x1="-86.36" y1="147.32" x2="-76.2" y2="147.32" width="0.1524" layer="91"/>
+<junction x="-86.36" y="147.32"/>
 </segment>
 <segment>
@@
 </segment>
 <segment>
-<pinref part="PROG" gate="G$1" pin="1"/>
-<wire x1="-45.72" y1="53.34" x2="-58.42" y2="53.34" width="0.1524" layer="91" grouprefs="PROGRAM"/>
-<label x="-55.88" y="53.34" size="1.778" layer="95" grouprefs="PROGRAM"/>
-</segment>
-<segment>
 <wire x1="20.32" y1="104.14" x2="35.56" y2="104.14" width="0.1524" layer="91" grouprefs="EXT-BUS"/>
 <label x="22.86" y="104.14" size="1.778" layer="95" grouprefs="EXT-BUS"/>
@@
 </segment>
 </net>
+<net name="EN" class="0">
+<segment>
+<pinref part="R5" gate="G$1" pin="1"/>
+<wire x1="-66.04" y1="147.32" x2="-50.8" y2="147.32" width="0.1524" layer="91"/>
+<wire x1="-50.8" y1="147.32" x2="-50.8" y2="142.24" width="0.1524" layer="91"/>
+<pinref part="U1" gate="G$1" pin="EN"/>
+<wire x1="-50.8" y1="142.24" x2="-45.72" y2="142.24" width="0.1524" layer="91"/>
+<wire x1="-50.8" y1="147.32" x2="-50.8" y2="152.4" width="0.1524" layer="91"/>
+<wire x1="-50.8" y1="152.4" x2="-63.5" y2="152.4" width="0.1524" layer="91"/>
+<junction x="-50.8" y="147.32"/>
+<label x="-60.96" y="152.4" size="1.778" layer="95"/>
+</segment>
+<segment>
+<pinref part="PROG" gate="G$1" pin="1"/>
+<wire x1="-45.72" y1="53.34" x2="-58.42" y2="53.34" width="0.1524" layer="91" grouprefs="PROGRAM"/>
+<label x="-55.88" y="53.34" size="1.778" layer="95" grouprefs="PROGRAM"/>
+</segment>
+</net>

Commit message: initial
Parts:
- removed COM: (no value), led:LEDCHIPLED_0603
- removed PROG: (no value), con-lstb:MA05-1
- added SV1: (no value), con-lstb:MA06-1
- added WIFI: LED_BLUE, Opto-Electronic:LED_CHIP_BLUE-1608
- 3,3V: value (none) -> LED_RED; device led:LEDCHIPLED_0603 -> Opto-Electronic:LED_CHIP_RED-1608
- 5V: value (none) -> LED_GREEN; device led:LEDCHIPLED_0603 -> Opto-Electronic:LED_CHIP_GREEN-1608
Connections:
- net +3V3: now also SV1.5; no longer PROG.4
- net EN: now also SV1.2; no longer PROG.1
- net GND: now also SV1.6, WIFI.C; no longer COM.C, PROG.5
- net IO0: now also SV1.1
- net N$3: now also WIFI.A; no longer COM.A
- net RXD0: now also SV1.3; no longer PROG.2
- net TXD0: now also SV1.4; no longer PROG.3
Other:
- moved on the sheet: C1, C10, C11, C12, C13, C7, IC1, IC2, R12, R4
